File: pe/buck_converter/buck_converter.kicad_sch (KiCad schematic)
At the start: 0 parts

Commit message: Simple Buck Circuit (no values or pwm)
Parts:
- added 12V_IN: 12V_IN, Package_DFN_QFN:QFN-40-1EP_6x6mm_P0.5mm_EP4.6x4.6mm, symbol Connector:Conn_01x02_Pin
- added 5V_OUT: (no value), Package_DFN_QFN:QFN-40-1EP_6x6mm_P0.5mm_EP4.6x4.6mm, symbol Connector:Conn_01x02_Pin
- added C1: C, symbol Device:C
- added D1: D, Diode_THT:D_DO-35_SOD27_P7.62mm_Horizontal, symbol Device:D
- added L1: L, Relay_THT:Relay_DPDT_Finder_30.22, symbol Device:L
- added Q1: BSS308PE, Package_TO_SOT_SMD:SOT-23_Handsoldering, symbol formula_slug_symbol_library:BSS308PE
Connections:
- new net: 12V_IN.1 (Pin_1), Q1.2 (S)
- new net: D1.1 (K), L1.1, Q1.3 (D)
- new net: 5V_OUT.1 (Pin_1), C1.1, L1.2
- new net GND: 12V_IN.2 (Pin_2), 5V_OUT.2 (Pin_2), C1.2, D1.2 (A)
