File: lv/kicad-template/template.kicad_sch (KiCad schematic)
At the start: 0 parts

Commit message: made template
Parts:
- added U1: AD8001AN, Package_DIP:DIP-8_W7.62mm, symbol Amplifier_Operational:AD8001AN
Connections:
- new net +3.3V: U1.7 (V+)
- new net GND: U1.4 (V-)
