File: lv/Kicad Projects/BSPD - Op Amp Comp/BSPD - Op Amp Comp.kicad_sch (KiCad schematic)
At the start: 3 parts, among them U1 MCP6004

Commit message: Labeling
Other:
- note added: "Basic Op-Amp Circuit"
- note removed: "ADC_CURRENT"
Changed lines of the file:
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@@
 		(comment 3 "${COMMENT2}")
 	)
-	(text "ADC_CURRENT"
+	(text "Basic Op-Amp Circuit\n"
 		(exclude_from_sim no)
-		(at 35.306 29.464 0)
+		(at 34.544 21.59 0)
 		(effects
 			(font
@@
 		)
 	)
+	(polyline
+		(pts
+			(xy 12.7 59.69) (xy 80.01 59.69)
+		)
+		(stroke
+			(width 0)
+			(type default)
+		)
+	)
 	(wire
 		(pts
@@
 		)
 		(stroke
+			(width 0)
+			(type default)
+		)
+	)
+	(polyline
+		(pts
+			(xy 80.01 12.7) (xy 80.01 59.69)
+		)
+		(stroke
