File: lv/Kicad Projects/FPC Strain Gauge/FPC Strain Gauge.kicad_sch (KiCad schematic)
At the start: 2 parts

Commit message: Labeling
Other:
- note added: "Use Copper Traces to act as an Resistor worth 350 ohms"
Changed lines of the file:
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@@
 		(comment 3 "${COMMENT2}")
+	)
+	(text "Use Copper Traces to act as an Resistor worth 350 ohms"
+		(exclude_from_sim no)
+		(at 48.26 35.052 0)
+		(effects
+			(font
+				(size 1.27 1.27)
+			)
+		)
 	)
 	(wire
