File: fs-5-schematics.kicad_pcb (KiCad board)
At the start: 2 copper layers, 0 parts

Commit message: erc+pcb attempt
Parts:
- added Cboost1: 0.1uF, Capacitor_SMD:C_0603_1608Metric_Pad1.08x0.95mm_HandSolder, F.Cu at (141.9, 70.0)
- added Cdecoupling1: 0.1uF, Capacitor_SMD:C_0603_1608Metric_Pad1.08x0.95mm_HandSolder, F.Cu at (115.9, 86.0)
- added Cfeedfoward1: 75pF, Capacitor_SMD:C_0603_1608Metric_Pad1.08x0.95mm_HandSolder, F.Cu at (153.9, 105.5)
- added Cinput1: 10uF, Capacitor_SMD:C_0805_2012Metric_Pad1.18x1.45mm_HandSolder, F.Cu at (108.0, 86.0)
- added Cout1: 22uF, Capacitor_SMD:C_0805_2012Metric_Pad1.18x1.45mm_HandSolder, F.Cu at (158.5, 79.5)
- added Cout2: 22uF, Capacitor_SMD:C_0805_2012Metric_Pad1.18x1.45mm_HandSolder, F.Cu at (168.0, 79.5)
- added L1: 10uH, Package_SON:WSON-8-1EP_6x5mm_P1.27mm_EP3.4x4mm, F.Cu at (150.7, 74.5)
- added R2: 100K, Resistor_SMD:R_0603_1608Metric_Pad0.98x0.95mm_HandSolder, F.Cu at (168.4, 105.5)
- added R3: 13.5K, Resistor_SMD:R_0603_1608Metric_Pad0.98x0.95mm_HandSolder, F.Cu at (167.0, 96.0)
- added R4: 510k, Resistor_SMD:R_0603_1608Metric_Pad0.98x0.95mm_HandSolder, F.Cu at (121.9, 72.5)
- added U1: TPS54202DDC, Package_TO_SOT_SMD:SOT-23-6, F.Cu at (131.9, 72.5)

Commit message: pcb + schm edit
Parts:
- moved Cfeedfoward1 19.0 mm to (146.4, 88.0), turned to 180 degrees
- moved Cboost1 16.9 mm to (130.5, 82.5)
- moved Cdecoupling1 8.13 mm to (120.0, 79.0)
- moved Cinput1 8.13 mm to (112.2, 79.0)
- moved L1 6.61 mm to (152.5, 68.2), turned to 90 degrees
- moved U1 5.00 mm to (130.0, 77.1), turned to 90 degrees
Other:
- board outline added: 79 x 50 mm

Commit message: PCb layouts complete?, need checked
Parts:
- added J1: 12V, TerminalBlock:TerminalBlock_MaiXu_MX126-5.0-02P_1x02_P5.00mm, F.Cu at (82.0, 67.0)
- added J2: 5V, TerminalBlock:TerminalBlock_MaiXu_MX126-5.0-02P_1x02_P5.00mm, F.Cu at (77.8, 39.0)
- moved Cout2 99.0 mm to (73.5, 49.8), turned to -90 degrees
- moved R2 90.1 mm to (96.1, 51.8), turned to 180 degrees
- moved Cout1 88.2 mm to (75.5, 49.8), turned to -90 degrees
- moved R3 81.7 mm to (96.1, 55.2)
- moved L1 74.1 mm to (80.0, 53.0), turned to 180 degrees
- moved Cfeedfoward1 61.0 mm to (96.1, 53.5)
- moved Cboost1 51.9 mm to (90.2, 49.8), turned to 180 degrees
- moved U1 47.1 mm to (90.0, 52.2), turned to 0 degrees
- moved Cdecoupling1 36.1 mm to (91.5, 56.9), turned to 90 degrees
- moved R4 34.0 mm to (96.2, 50.2), turned to 180 degrees
- moved Cinput1 31.7 mm to (89.5, 56.9), turned to 90 degrees
Connections:
- Cfeedfoward1 pad 1: Net-(U1-FB) -> +5V
- Cfeedfoward1 pad 2: GND -> Net-(U1-FB)
- Cout1 pad 1: Net-(J2-Pin_2) -> +5V
- Cout2 pad 1: Net-(J2-Pin_2) -> +5V
- L1 pad 2: Net-(J2-Pin_2) -> +5V
- R2 pad 1: Net-(U1-FB) -> +5V
- R2 pad 2: GND -> Net-(U1-FB)
- R3 pad 1: Net-(J2-Pin_2) -> Net-(U1-FB)
- R3 pad 2: Net-(U1-FB) -> GND
Routing:
- net +5V: track 0.00 -> 48.8 mm
- net +12V: track 0.00 -> 42.5 mm
- net GND: track 0.00 -> 32.7 mm, vias 0 -> 2
- net Net-(U1-SW): track 0.00 -> 15.2 mm
- net Net-(U1-FB): track 0.00 -> 8.35 mm
- net Net-(U1-EN): track 0.00 -> 5.44 mm
- net Net-(U1-BOOT): track 0.00 -> 1.56 mm
- added copper zone on B.Cu, net GND
- added copper zone on F.Cu, net GND
Other:
- board size 79 x 50 mm -> 34 x 36.8 mm
