File: fs-5-schematics.kicad_sch (KiCad schematic)
At the start: 13 parts, among them J1 12V, J2 5V, U1 TPS54202DDC

Commit message: added all footprints + google doc link
Parts:
- Cboost1, Cdecoupling1, Cfeedfoward1: footprint (none) -> Capacitor_SMD:C_0603_1608Metric_Pad1.08x0.95mm_HandSolder
- Cinput1, Cout1, Cout2: footprint (none) -> Capacitor_SMD:C_0805_2012Metric_Pad1.18x1.45mm_HandSolder
- R2, R3: footprint 0603 -> Resistor_SMD:R_0603_1608Metric_Pad0.98x0.95mm_HandSolder
- R4: footprint (none) -> Resistor_SMD:R_0603_1608Metric_Pad0.98x0.95mm_HandSolder
Other:
- note added: "Google Doc Link"
Changed lines of the file:
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@@
 		(comment 3 "${COMMENT2}")
+	)
+	(text "Google Doc Link"
+		(exclude_from_sim no)
+		(at 125.476 197.612 0)
+		(effects
+			(font
+				(size 5.08 5.08)
+			)
+			(href "https://docs.google.com/document/d/1l8F47zrDbMXuP6yOvAKSnpXGTaubscwsjH4vZ9yr-mc/edit?tab=t.b8f5retqd1r")
+		)
 	)
 	(junction
@@
 			)
 		)
-		(property "Footprint" ""
+		(property "Footprint" "Capacitor_SMD:C_0805_2012Metric_Pad1.18x1.45mm_HandSolder"
 			(at 82.2452 102.87 0)
 			(hide yes)
@@
 			)
 		)
-		(property "Footprint" ""
+		(property "Footprint" "Capacitor_SMD:C_0805_2012Metric_Pad1.18x1.45mm_HandSolder"
 			(at 177.4952 88.9 0)
 			(hide yes)
@@
 			)
 		)
-		(property "Footprint" "0603"
+		(property "Footprint" "Resistor_SMD:R_0603_1608Metric_Pad0.98x0.95mm_HandSolder"
 			(at 209.042 105.41 90)
 			(hide yes)
@@
 			)
 		)
-		(property "Footprint" ""
+		(property "Footprint" "Capacitor_SMD:C_0603_1608Metric_Pad1.08x0.95mm_HandSolder"
 			(at 100.0252 102.87 0)
 			(hide yes)
@@
 			)
 		)
-		(property "Footprint" ""
+		(property "Footprint" "Capacitor_SMD:C_0603_1608Metric_Pad1.08x0.95mm_HandSolder"
 			(at 160.02 71.4248 0)
 			(hide yes)
@@
 			)
 		)
-		(property "Footprint" ""
+		(property "Footprint" "Capacitor_SMD:C_0805_2012Metric_Pad1.18x1.45mm_HandSolder"
 			(at 188.9252 88.9 0)
 			(hide yes)
@@
 			)
 		)
-		(property "Footprint" ""
+		(property "Footprint" "Resistor_SMD:R_0603_1608Metric_Pad0.98x0.95mm_HandSolder"
 			(at 112.522 80.01 90)
 			(hide yes)
@@
 			)
 		)
-		(property "Footprint" "0603"
+		(property "Footprint" "Resistor_SMD:R_0603_1608Metric_Pad0.98x0.95mm_HandSolder"
 			(at 209.042 93.98 90)
 			(hide yes)
@@
 			)
 		)
-		(property "Footprint" ""
+		(property "Footprint" "Capacitor_SMD:C_0603_1608Metric_Pad1.08x0.95mm_HandSolder"
 			(at 191.4652 109.22 0)
 			(hide yes)

Commit message: erc+pcb attempt
Connections:
- net GND: now also J2.1 (Pin_1)
- net +12V: now reaches Cdecoupling1.1, Cinput1.1, J1.1 (Pin_1), R4.1, U1.3 (VIN)
- net +5V: now reaches Cout1.1, Cout2.1, J2.2 (Pin_2), L1.2, R3.1

Commit message: pcb + schm edit
Changed lines of the file:
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@@
+	)
+	(junction
+		(at 63.5 76.2)
+		(diameter 0)
+		(color 0 0 0 0)
 	)
 	(junction
@@
 	)
 	(junction
-		(at 220.98 81.28)
-		(diameter 0)
-		(color 0 0 0 0)
-	)
-	(junction
 		(at 81.28 76.2)
 		(diameter 0)
@@
 		(color 0 0 0 0)
 	)
-	(junction
-		(at 63.5 87.63)
-		(diameter 0)
-		(color 0 0 0 0)
-	)
 	(wire
 		(pts
@@
 	(wire
 		(pts
-			(xy 63.5 87.63) (xy 63.5 97.79)
+			(xy 63.5 78.74) (xy 63.5 97.79)
 		)
 		(stroke
@@
 	(wire
 		(pts
-			(xy 220.98 81.28) (xy 232.41 81.28)
-		)
-		(stroke
-			(width 0)
-			(type default)
-		)
-	)
-	(wire
-		(pts
 			(xy 114.3 76.2) (xy 127 76.2)
 		)
@@
 	(wire
 		(pts
-			(xy 210.82 81.28) (xy 220.98 81.28)
+			(xy 210.82 81.28) (xy 232.41 81.28)
 		)
 		(stroke
@@
 		(pts
 			(xy 99.06 95.25) (xy 99.06 76.2)
-		)
-		(stroke
-			(width 0)
-			(type default)
-		)
-	)
-	(wire
-		(pts
-			(xy 63.5 78.74) (xy 63.5 87.63)
 		)
 		(stroke
@@
 	(symbol
 		(lib_id "power:+5V")
-		(at 220.98 81.28 270)
+		(at 210.82 81.28 0)
 		(unit 1)
 		(body_style 1)
@@
 		(fields_autoplaced yes)
 		(property "Reference" "#PWR06"
-			(at 217.17 81.28 0)
+			(at 210.82 85.09 0)
 			(hide yes)
 			(show_name no)
@@
 		)
 		(property "Value" "+5V"
-			(at 224.79 81.2799 90)
+			(at 213.36 80.0099 0)
 			(show_name no)
 			(do_not_autoplace no)
@@
 		)
 		(property "Footprint" ""
-			(at 220.98 81.28 0)
+			(at 210.82 81.28 0)
 			(hide yes)
 			(show_name no)
@@
 		)
 		(property "Datasheet" ""
-			(at 220.98 81.28 0)
+			(at 210.82 81.28 0)
 			(hide yes)
 			(show_name no)
@@
 		)
 		(property "Description" "Power symbol creates a global label with name \"+5V\""
-			(at 220.98 81.28 0)
+			(at 210.82 81.28 0)
 			(hide yes)
 			(show_name no)
@@
 	(symbol
 		(lib_id "power:+12V")
-		(at 63.5 87.63 0)
+		(at 63.5 76.2 0)
 		(unit 1)
 		(body_style 1)
@@
 		(fields_autoplaced yes)
 		(property "Reference" "#PWR05"
-			(at 63.5 91.44 0)
+			(at 63.5 80.01 0)
 			(hide yes)
 			(show_name no)
@@
 		)
 		(property "Value" "+12V"
-			(at 63.5 82.55 0)
+			(at 63.5 71.12 0)
 			(show_name no)
 			(do_not_autoplace no)
@@
 		)
 		(property "Footprint" ""
-			(at 63.5 87.63 0)
+			(at 63.5 76.2 0)
 			(hide yes)
 			(show_name no)
@@
 		)
 		(property "Datasheet" ""
-			(at 63.5 87.63 0)
+			(at 63.5 76.2 0)
 			(hide yes)
 			(show_name no)
@@
 		)
 		(property "Description" "Power symbol creates a global label with name \"+12V\""
-			(at 63.5 87.63 0)
-			(hide yes)
-			(show_name no)
+			(at 63.5 76.2 0)
+			(hide yes)
+			(show_name no)

Commit message: PCb layouts complete?, need checked
Parts:
- J1, J2: footprint (none) -> TerminalBlock:TerminalBlock_MaiXu_MX126-5.0-02P_1x02_P5.00mm
Connections:
- net +5V: now also Cfeedfoward1.1, R2.1; no longer R3.1
- net GND: now also R3.2; no longer Cfeedfoward1.2, R2.2
- new net: Cfeedfoward1.2, R2.2, R3.1, U1.4 (FB)
Other:
- moved on the sheet: Cfeedfoward1, R2
