File: pe/Buck-Converter-Design/template.kicad_sch (KiCad schematic)
At the start: 7 parts, among them U1 TPS562200

Commit message: LV notes Op Amps
How they work and what they are used for
Other:
- title: ${BOARD_TITLE} -> Buck Converter
Changed lines of the file:
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@@
 	(paper "A")
 	(title_block
-		(title "${BOARD_TITLE}")
+		(title "Buck Converter")
 		(date "${CURRENT_DATE}")
 		(rev "${REVISION}")
 		(company "Formula Slug")
-		(comment 1 "${NAMES}")
+		(comment 1 "Jackson Pesmark")
 		(comment 2 "${COMMENT1}")
 		(comment 3 "${COMMENT2}")
