File: lv/BMS PCB ONBOARDING.kicad_sch (KiCad schematic)
At the start: 42 parts, among them J1 84952-5, J2 84952-5, J3 512810598, J3_B12_POWER1 84952-5, J4 1053131202, J5 512810598, J6 1053131202, J7 1053131202, J8 1053131202, Q1 NSV1C201MZ4, SW1 SW_DIP_x04, U3 LTC6811IG-2-TRPBF

Commit message: UPDATE 2: LTC6811 -> BQ79616
FS-6: BQ79616 bring-up — all 65 pins assigned, blocks checked and fixed

Chip wiring:
- Cell ladder VC0–VC16 placed
- Supply caps checked against a TI design review — DVDD was originally 1uF,
  now changed to be 2.2uF
- EPAD (pin 65) wired to GND on its own leg 
- Ground pins AVSS/CVSS/DVSS each get their own leg to a GND symbol
- BAT filter placed
- GPIO1 = I2C_SDA, GPIO2 = I2C_SCL, GPIO3 = ALERT, GPIO4 = DQ used for TEMP
- GPIO5–8: one 10k to GND each 
- BBP/BBN left NC 
- RX/TX left NC 

Blocks on the sheet:
- Temp pull-ups changed from VREG to TSREF 
- COM ports ×4 kept — coupling caps, chokes, TVS, 0Ω links all checked
- J701/J702 option connectors: removed NC flags, marked DNP
- 9 test points kept, NC flags removed 
- NPN power block: probably going to delete not needed as a result
   of BQ79616 inner power source TSREF

Learned: 
-the BQ79616 makes its own power. Unlike the old chip family,
  it generates its internal supply rails (AVDD, CVDD, DVDD, TSREF) 
-no external regulator or regulator circuit needed. This also means
 different parts of the chip run at different voltages, so each rail needs
 its own decoupling cap, sized from the datasheet. 
- verify part values against datasheet that is the main reason the 
   DVDD mistake was caught.
Parts:
- removed C1: 10nF, Capacitor_SMD:C_0805_2012Metric_Pad1.18x1.45mm_HandSolder, symbol Device:C
- removed C2, C6: 100nF, Capacitor_SMD:C_0805_2012Metric_Pad1.18x1.45mm_HandSolder, symbol Device:C
- removed C3, C4, C5: 1uF, Capacitor_SMD:C_0805_2012Metric_Pad1.18x1.45mm_HandSolder, symbol Device:C
- removed C7: 15pF, Capacitor_SMD:C_0805_2012Metric_Pad1.18x1.45mm_HandSolder, symbol Device:C
- removed C8: 10nF, Capacitor_SMD:C_0805_2012Metric_Pad1.18x1.45mm_HandSolder, symbol Device:C_Small
- removed D1, D2: LH R974-LP-1, LED_SMD:LED_0805_2012Metric_Pad1.15x1.40mm_HandSolder, symbol Device:LED_Small
- removed J1, J2, J3_B12_POWER1: 84952-5, FS_4_Global_Footprint_Library:849525, symbol Connector_Generic:Conn_01x05
- removed J7, J8: 1053131202, FS_4_Global_Footprint_Library:Nano-Fit_1054301102, symbol Connector:Conn_01x02_Pin
- removed L1: HM2113ZNLT, FS_4_Global_Footprint_Library:HM2113ZNLT, symbol FS_4_Global_Symbol_Library:HM2113ZNLT
- removed Q1: NSV1C201MZ4, Package_TO_SOT_SMD:SOT-223, symbol Device:Q_NPN_BCEC
- removed R10, R11, R13: 10k, Resistor_SMD:R_0805_2012Metric_Pad1.20x1.40mm_HandSolder, symbol Device:R
- removed R15, R16: 22, Resistor_SMD:R_0805_2012Metric_Pad1.20x1.40mm_HandSolder, symbol Device:R
- removed R17: 200, Resistor_SMD:R_0805_2012Metric_Pad1.20x1.40mm_HandSolder, symbol Device:R_Small
- removed R3, R5: 160, Resistor_SMD:R_0805_2012Metric_Pad1.20x1.40mm_HandSolder, symbol Device:R_Small
- removed R6: 1.5k, Resistor_SMD:R_0805_2012Metric_Pad1.20x1.40mm_HandSolder, symbol Device:R
- removed SW1: SW_DIP_x04, FS_4_Global_Footprint_Library:SW_A6H-4101_OMR, symbol Switch:SW_DIP_x04
- removed U3: LTC6811IG-2-TRPBF, FS_3_Global_Footprint_Library:LTC6811-2, symbol FS_3_Global_Symbol_Library:LTC6811IG-2-TRPBF
- added C201: 10nF, GCM188R72A103KA37J:CAPC1608X90N, symbol GCM188R72A103KA37J:GCM188R72A103KA37J
- added C202, C208: 0.1uF, GCM155R71A104KA55D:CAP_GCM15_1p05X0p55X0p55_MUR-L, symbol GCM155R71A104KA55D:GCM155R71A104KA55D
- added C203, C205, C210: 1uF, C0603C105K8RACAUTO:CAPC18095_95N_KEM-L, symbol C0603C105K8RACAUTO:C0603C105K8RACAUTO
- added C207: 2.2.uF, C0603C105K8RACAUTO:CAPC18095_95N_KEM-L, symbol C0603C105K8RACAUTO:C0603C105K8RACAUTO
- added C209: 4.7uF, C2012X7R1A475M125AC:CAP_2012_TDK-L, symbol C2012X7R1A475M125AC:C2012X7R1A475M125AC
- added C601: 0.22uF, GCM31MR72A224KA37L:G-31_MUR-L, symbol GCM31MR72A224KA37L:GCM31MR72A224KA37L
- added C701, C702, C707, C708: 2200pF, 1206J2K00222KXR (1):CAPC3216X160N, symbol 1206J2K00222KXR:1206J2K00222KXR
- added C703, C704, C705, C706: 220pF, CL10B221JB8NNNC:CAP_CL10_SAM-L, symbol CL10B221JB8NNNC:CL10B221JB8NNNC
- added D701, D702: 24V, Package_TO_SOT_SMD:SOT-23, symbol PESD1CAN,215:PESD1CAN_215
- added FL701, FL702: 470uH, KiCad:744242471, symbol 744242471:744242471
- added J701, J702: 430450200, 0430450200:CON_430450200_MOL, symbol 0430450200:430450200
- added Q601: ZXTN4004KTC, ZXTN4004KTC:ZXTN4004KTC, symbol ZXTN4004KTC:ZXTN4004KTC
- added R201: 30, ERJ-3EKF30R0V:RC0603N_PAN-L, symbol 2024-10-08_19-57-08:ERJ-3EKF30R0V
- added R3: 10k, symbol Device:R
- added R5: 5k, symbol Device:R
- added R601: 100, CRCW2010100RFKEF:RES_CRCW_2010-L, symbol CRCW2010100RFKEF:CRCW2010100RFKEF
- added R602: 200, Resistor_SMD:R_2512_6332Metric, symbol CRCW2010200RFKEF:CRCW2010200RFKEF
- added R701, R702, R705, R706, R709, R710, R713, R714, R715, R716, R721, R722: 0, CRCW08050000Z0EAHP:RES_CRCW_0805_VIS-L, symbol CRCW08050000Z0EAHP:CRCW08050000Z0EAHP
- added R703, R704, R719, R720: 0, RC0603JR-070RL:RC0603N_YAG-L, symbol RC0603JR-070RL:RC0603JR-070RL
- added R707, R708, R717, R718: 51, CRCW060351R0JNEA:RC0603N_VIS-L, symbol CRCW060351R0JNEA:CRCW060351R0JNEA
- added R711, R712: 1k, ERJ-3EKF1001V:RC0603N_PAN-L, symbol ERJ-3EKF1001V:ERJ-3EKF1001V
- added TP501, TP502, TP503, TP504, TP505, TP506, TP507, TP508, TP509: 5012, 5012:TP_5012, symbol 5012:5012
- added U1: BQ79616PAPRQ1, PAP0064F-IPC_A, symbol 2026-10-08_21-00-57:BQ79616PAPRQ1
- R1, R4: value 100 -> 10k; footprint Resistor_SMD:R_0805_2012Metric_Pad1.20x1.40mm_HandSolder -> (none); Digi PN 311-100CRCT-ND -> (none); Digi URL https://www.digikey.com/en/products/detail/yageo/RC0805FR-0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 -> (none); MFG YAGEO -> (none); MFG PN RC0805FR-07100RL -> (none)
- R2: value 10 -> 10k; footprint Resistor_SMD:R_0805_2012Metric_Pad1.20x1.40mm_HandSolder -> (none); Digi PN 13-RC0805FR-1010RLCT-ND -> (none); Digi URL https://www.digikey.com/en/products/detail/yageo/RC0805FR-1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 -> (none); MFG YAGEO -> (none); MFG PN RC0805FR-1010RL -> (none)
- R7: value 680 -> 5k; footprint Resistor_SMD:R_0805_2012Metric_Pad1.20x1.40mm_HandSolder -> (none); Digi PN 311-680CRCT-ND -> (none); Digi URL https://www.digikey.com/en/products/detail/yageo/RC0805FR-0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 -> (none); MFG YAGEO -> (none); MFG PN RC0805FR-07680RL -> (none)
- R8: value 402 -> 5k; footprint Resistor_SMD:R_0805_2012Metric_Pad1.20x1.40mm_HandSolder -> (none); Digi PN 13-AC0805FR-07402RLCT-ND -> (none); Digi URL https://www.digikey.com/en/products/detail/yageo/AC0805FR-0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 -> (none); MFG YAGEO -> (none); MFG PN AC0805FR-07402RL -> (none)
Connections:
- net BB0/B# is gone; now on net GND: R1.2
- net ICMP is gone; now on net I2C_SDA: R7.2
- net ALERT: now also R5.2, U1.59 (GPIO3)
- net DQ: now also U1.58 (GPIO4)
- net I2C_SCL: now also R8.2, U1.60 (GPIO2)
- net I2C_SDA: now also U1.61 (GPIO1)
- net V-: no longer R7.1
- net VREG: no longer J3.5 (Pin_5)
- net at R2.1: now also U1.55 (GPIO7)
- net GND: now reaches R2.2, R4.2
- net GND: now also C201.1, C202.1, C203.1, C205.1, C207.1, C208.1, C209.1, C210.1, C601.2, C703.1, C704.1, C705.1, C706.1, D701.3, D702.3, R3.2, U1.36 (REFHM), U1.39 (AVSS), U1.46 (CVSS), U1.50 (DVSS), U1.65 (PAD)
- net at R4.1: now also U1.56 (GPIO6)
- net BB6/S#+1: no longer names the net of R43.1
- net C0: no longer names the net of R1.1
- net C0: now also U1.54 (GPIO8)
- net IsoSPI_P renamed TSREF
- net TSREF: now also J3.5 (Pin_5), R7.1, C205.2, R5.1, TP502.TP, U1.51 (TSREF)
- net S7: no longer names the net of R43.2
- net S7: no longer TP1.1
- new net: C701.1, FL701.4 (N1-), R705.1
- new net: C701.2, R709.2
- new net: C708.1, FL702.3 (N2-), R716.1
- new net: FL702.2 (N2+), R716.2, R722.1
- new net: C601.1, Q601.2 (C), R601.2
- new net: C707.1, FL702.4 (N1-), R715.1
- new net: FL702.1 (N1+), R715.2, R721.1
- new net: D701.2, R704.2, R707.2
- new net: C702.2, R710.2
- new net: C702.1, FL701.3 (N2-), R706.1
- new net: FL701.1 (N1+), R701.1, R705.2
- new net: D702.2, R718.2, R720.2
- new net: R601.1, R602.1
- new net: FL701.2 (N2+), R702.1, R706.2
- new net: C708.2, R714.2
- new net: D702.1, R717.2, R719.2
- new net: C707.2, R713.2
- new net: C201.2, R201.1, U1.1 (BAT)
- new net: D701.1, R703.2, R708.2
- new net: R3.1, U1.57 (GPIO5)
- new net AVDD: C210.2, TP505.TP, U1.38 (AVDD)
- new net BAT: R201.2, U1.3 (VC16)
- new net CB0: U1.34 (CB0)
- new net CB1: U1.32 (CB1)
- new net CB10: U1.14 (CB10)
- new net CB11: U1.12 (CB11)
- new net CB12: U1.10 (CB12)
- new net CB13: U1.8 (CB13)
- new net CB14: U1.6 (CB14)
- new net CB15: U1.4 (CB15)
- new net CB16: U1.2 (CB16)
- new net CB2: U1.30 (CB2)
- new net CB3: U1.28 (CB3)
- new net CB4: U1.26 (CB4)
- new net CB5: U1.24 (CB5)
- new net CB6: U1.22 (CB6)
- new net CB7: U1.20 (CB7)
- new net CB8: U1.18 (CB8)
- new net CB9: U1.16 (CB9)
- new net COMHN: C705.2, R712.1, R718.1, U1.42 (COMHN)
- new net COMHP: C706.2, R712.2, R717.1, U1.43 (COMHP)
- new net COMLN: C703.2, R708.1, R711.1, U1.41 (COMLN)
- new net COMLP: C704.2, R707.1, R711.2, U1.40 (COMLP)
- new net COMMH_N_OPT-: R713.1, R720.1
- new net COMMH_P_OPT+: R714.1, R719.1
- new net COMML_N_OPT-: R703.1, R710.1
- new net COMML_P_OPT+: R704.1, R709.1
- new net CVDD: C209.2, TP503.TP, U1.45 (CVDD)
- new net Cell 14: R602.2
- new net DVDD: C207.2, TP501.TP, U1.49 (DVDD)
- new net ISO_COMMH_N: J702.2, R721.2
- new net ISO_COMMH_P: J702.1, R722.2
- new net ISO_COMML_N: J701.1, R702.2
- new net ISO_COMML_P: J701.2, R701.2
- new net LDOIN: C208.2, Q601.3 (E), TP504.TP, U1.47 (LDOIN)
- new net NEG5V: C202.2, TP506.TP, U1.44 (NEG5V)
- new net NFAULT: TP508.TP, U1.62 (FAULT_N)
- new net NPNB: Q601.1 (B), TP509.TP, U1.48 (NPNB)
- new net REFHP: C203.2, TP507.TP, U1.37 (REFHP)
- new net VC0: U1.35 (VC0)
- new net VC1: U1.33 (VC1)
- new net VC10: U1.15 (VC10)
- new net VC11: U1.13 (VC11)
- new net VC12: U1.11 (VC12)
- new net VC13: U1.9 (VC13)
- new net VC14: U1.7 (VC14)
- new net VC15: U1.5 (VC15)
- new net VC2: U1.31 (VC2)
- new net VC3: U1.29 (VC3)
- new net VC4: U1.27 (VC4)
- new net VC5: U1.25 (VC5)
- new net VC6: U1.23 (VC6)
- new net VC7: U1.21 (VC7)
- new net VC8: U1.19 (VC8)
- new net VC9: U1.17 (VC9)
Other:
- removed sheet BB0
- removed sheet BB1
- removed sheet BB10
- removed sheet BB11
- removed sheet BB2
- removed sheet BB3
- removed sheet BB4
- removed sheet BB5
- removed sheet BB6
- removed sheet BB7
- removed sheet BB8
- removed sheet BB9
- note removed: "1: ISOSpi Termintion 2: Address bit 2 3: Address bit 1 4: Address bit 0"
- note removed: "Bottom filtering not caught by BalanceSenseBlock"
- note removed: "Configuration-specific settings switches"
- note removed: "ISOSpi Bias setting"
- note removed: "ISOSpi isolation and filtering"
- note removed: "LTC6810 (6-cell) → LTC6811IG-2-TRPBF (12-cell) Learned: cells-per-chip reshapes the pack and add fully different architecture • Double the capacity: Monitors up to 12 series cells instead of 6, cutting the required number of ICs and components in half. • Higher precision: Drops maximum measurement error from 1.8 mV to 1.2 mV, which is critical for flat-voltage chemistries like LiFePO4. • Faster t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"
- note removed: "This module was designed as specified in the LTC6811 datasheet."
