File: pe/kicad-template/template.kicad_sch (KiCad schematic)
At the start: 0 parts

Commit message: Working on schematic. Uploaded notes for Act1.
Parts:
- added C1: 15uF, Capacitor_SMD:C_0603_1608Metric, symbol Device:C_Small
- added L1: 10.5uH, Inductor_SMD:L_0603_1608Metric, symbol Device:L_Small
- added R1: R_Load, symbol Device:R_Small
- added U1: (no value), Package_TO_SOT_SMD:SOT-23-6, symbol Custom_Library:TPS542025DDCR
Connections:
- new net: L1.1, U1.2 (SW)
- new net: C1.1, L1.2, R1.1
- new net GND: C1.2, R1.2, U1.1 (GND)
- new net V_in 13.5v: U1.3 (VIN)
