File: pe/kicad-template/template.kicad_sch (KiCad schematic)
At the start: 0 parts

Commit message: Everything seems complete
Parts:
- added BuckIC1: AP63205WU, Package_TO_SOT_SMD:TSOT-23-6, symbol Regulator_Switching:AP63205WU
- added C1: 10UF, Capacitor_SMD:C_0603_1608Metric, symbol Device:C
- added C2: 22UF, Capacitor_SMD:C_0603_1608Metric, symbol Device:C
- added C3: 100nF, Capacitor_SMD:C_0603_1608Metric, symbol Device:C
- added L1: 4.7UH, Inductor_SMD:L_Bourns_SRP5030T, symbol Device:L
Connections:
- new net: BuckIC1.5 (SW), C3.2, L1.1
- new net: BuckIC1.6 (BST), C3.1
- new net +15V: BuckIC1.2 (EN), BuckIC1.3 (IN), C1.1
- new net +5V: BuckIC1.1 (FB), C2.1, L1.2
- new net GND: BuckIC1.4 (GND), C1.2, C2.2
