File: lv/workshop/workshop.kicad_sch (KiCad schematic)
At the start: 0 parts

Commit message: Updated ETC controller and KiCad workshop stuff
Parts:
- added C1: C_Small, Connector:Banana_Cliff_FCR7350N_S16N-PC_Horizontal, symbol Device:C_Small
- added D1: D, Diode_SMD:D_1210_3225Metric, symbol Device:D
- added J2, J3: Conn_01x02, Connector_RJ:RJ45_Abracon_ARJP11A-MA_Horizontal, symbol Connector_Generic:Conn_01x02
- added R1: 24k, Resistor_SMD:R_Array_Convex_4x0612, symbol Device:R_Small
- added R2: 1k, Connector_AMASS:AMASS_XT60-M_1x02_P7.20mm_Vertical, symbol Device:R_Small
- added U1: MCP6004, Package_SO:SOIC-14_3.9x8.7mm_P1.27mm, symbol Amplifier_Operational:MCP6004
Connections:
- new net: R1.2, R2.1, U1.3 (+)
- new net: J3.2 (Pin_2), U1.6 (-), U1.7
- new net: J2.2 (Pin_2), R1.1
- new net: D1.2 (A), U1.1
- new net: C1.1, D1.1 (K), U1.2 (-), U1.5 (+)
- new net GND: C1.2, J2.1 (Pin_1), J3.1 (Pin_1), R2.2
