File: pe/Buck_Conv/Buck_Conv.kicad_sch (KiCad schematic)
At the start: 11 parts, among them U1 BD95821MUV-E2

Commit message: buck converter annotations
Parts:
- C1, C2: value C_Small -> 10microF
- C3, C4: value C_Small -> 22microF
- C5: value C_Small -> 10nF
- C6: value C_Small -> 22nF
- L1: value L_Small -> 3.3microH
- R1: value R_Small -> 13kOhms
- R2: value R_Small -> 1.5kOhms
- R3: value R_Small -> 4.7kOHms
Connections:
- net GND: now also U1.10 (PGOOD)
