File: lv/Amay-Singhania/adc_with_pga.kicad_sch (KiCad schematic)
At the start: 6 parts, among them SW3 SW_DIP_x04, SW4 SW_DIP_x02, U4 ADS122C14IRTER

Commit message: Updated PCB with RC values for low pass filter. has old onboarding sheets with in-Amp and other designs, will be removed in next commit
Parts:
- C15: renamed from C11; footprint Package_TO_SOT_SMD:TSOT-23-5 -> Capacitor_SMD:C_0402_1005Metric
- C16: renamed from C12; footprint Package_TO_SOT_SMD:TSOT-23-5 -> Capacitor_SMD:C_0402_1005Metric
- C17: renamed from C13; footprint Package_TO_SOT_SMD:TSOT-23-5 -> Capacitor_SMD:C_0402_1005Metric
- SW5: renamed from SW3; footprint (none) -> Button_Switch_SMD:SW_DIP_SPSTx04_Slide_6.7x11.72mm_W6.73mm_P2.54mm_LowProfile_JPin
- SW6: renamed from SW4; footprint (none) -> Button_Switch_SMD:SW_DIP_SPSTx02_Slide_6.7x6.64mm_W6.73mm_P2.54mm_LowProfile_JPin
- renumbered U4 to U5
Connections:
- net +IN Center Axial Gauge renamed +IN Center_Gauge
- net +IN Left Axial Gauge renamed +IN Left_Gauge
- net +IN Right Axial Gauge renamed +IN Right_Gauge
- net -IN Center Axial Gauge renamed -IN Center_Gauge
- net -IN Left Axial Gauge renamed -IN Left_Gauge
- net -IN Right Axial Gauge renamed -IN Right_Gauge
- net ADC SCL renamed ADC_SCL
- net ADC SDA renamed ADC_SDA
Changed lines of the file:
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@@
 		)
 	)
-	(global_label "+IN Left Axial Gauge"
+	(global_label "+IN Left_Gauge"
 		(shape input)
 		(at 55.88 74.93 180)
@@
 		)
 	)
-	(global_label "ADC SDA"
+	(global_label "ADC_SDA"
 		(shape bidirectional)
 		(at 81.28 106.68 270)
@@
 		)
 	)
-	(global_label "+IN Center Axial Gauge"
+	(global_label "+IN Center_Gauge"
 		(shape input)
 		(at 55.88 69.85 180)
@@
 		)
 	)
-	(global_label "-IN Right Axial Gauge"
+	(global_label "-IN Right_Gauge"
 		(shape input)
 		(at 55.88 67.31 180)
@@
 		)
 	)
-	(global_label "-IN Center Axial Gauge"
+	(global_label "-IN Center_Gauge"
 		(shape input)
 		(at 55.88 72.39 180)
@@
 		)
 	)
-	(global_label "+IN Right Axial Gauge"
+	(global_label "+IN Right_Gauge"
 		(shape input)
 		(at 55.88 64.77 180)
@@
 		)
 	)
-	(global_label "ADC SDA"
+	(global_label "ADC_SDA"
 		(shape bidirectional)
 		(at 124.46 57.15 0)
@@
 		)
 	)
-	(global_label "ADC SCL"
+	(global_label "ADC_SCL"
 		(shape output)
 		(at 78.74 106.68 270)
@@
 		)
 	)
-	(global_label "ADC SCL"
+	(global_label "ADC_SCL"
 		(shape input)
 		(at 124.46 54.61 0)
@@
 		)
 	)
-	(global_label "-IN Left Axial Gauge"
+	(global_label "-IN Left_Gauge"
 		(shape input)
 		(at 55.88 77.47 180)
@@
 		(in_pos_files yes)
 		(dnp no)
-		(property "Reference" "C12"
+		(property "Reference" "C16"
 			(at 44.196 47.752 0)
 			(show_name no)
@@
 			)
 		)
-		(property "Footprint" "Package_TO_SOT_SMD:TSOT-23-5"
+		(property "Footprint" "Capacitor_SMD:C_0402_1005Metric"
 			(at 51.1048 44.45 0)
 			(hide yes)
@@
 			(project "Amay-Singhania"
 				(path "/94d2054e-a50f-482d-afff-dfa6248d499c"
-					(reference "C12")
+					(reference "C16")
 					(unit 1)
 				)
@@
 		(dnp no)
 		(fields_autoplaced yes)
-		(property "Reference" "U4"
+		(property "Reference" "U5"
 			(at 90.17 39.37 0)
 			(show_name no)
@@
 			(project "Amay-Singhania"
 				(path "/94d2054e-a50f-482d-afff-dfa6248d499c"
-					(reference "U4")
+					(reference "U5")
 					(unit 1)
 				)
@@
 		(in_pos_files yes)
 		(dnp no)
-		(property "Reference" "C11"
+		(property "Reference" "C15"
 			(at 40.386 35.052 0)
 			(show_name no)
@@
 			)
 		)
-		(property "Footprint" "Package_TO_SOT_SMD:TSOT-23-5"
+		(property "Footprint" "Capacitor_SMD:C_0402_1005Metric"
 			(at 47.2948 31.75 0)
 			(hide yes)
@@
 			(project "Amay-Singhania"
 				(path "/94d2054e-a50f-482d-afff-dfa6248d499c"
-					(reference "C11")
+					(reference "C15")
 					(unit 1)
 				)
@@
 		(dnp no)
 		(fields_autoplaced yes)
-		(property "Reference" "SW4"
+		(property "Reference" "SW6"
 			(at 110.49 97.7899 90)
 			(show_name no)
@@
 			)
 		)
-		(property "Footprint" ""
+		(property "Footprint" "Button_Switch_SMD:SW_DIP_SPSTx02_Slide_6.7x6.64mm_W6.73mm_P2.54mm_LowProfile_JPin"
 			(at 104.14 99.06 0)
 			(hide yes)
@@
 			(project "Amay-Singhania"
 				(path "/94d2054e-a50f-482d-afff-dfa6248d499c"
-					(reference "SW4")
+					(reference "SW6")
 					(unit 1)
 				)
@@
 		(in_pos_files yes)
 		(dnp no)
-		(property "Reference" "#PWR040"
+		(property "Reference" "#PWR061"
 			(at 143.51 49.53 0)
 			(hide yes)
@@
 			(project "Amay-Singhania"
 				(path "/94d2054e-a50f-482d-afff-dfa6248d499c"
-					(reference "#PWR040")
+					(reference "#PWR061")
 					(unit 1)
 				)
@@
 		(in_pos_files yes)
 		(dnp no)
-		(property "Reference" "#PWR036"
+		(property "Reference" "#PWR057"
 			(at 104.14 102.87 0)
 			(hide yes)
@@
 			(project "Amay-Singhania"
 				(path "/94d2054e-a50f-482d-afff-dfa6248d499c"
-					(reference "#PWR036")
+					(reference "#PWR057")
 					(unit 1)
 				)
@@
 		(in_pos_files yes)
 		(dnp no)
-		(property "Reference" "#PWR038"
+		(property "Reference" "#PWR060"
 			(at 135.89 74.93 0)
 			(hide yes)
@@
 			(project "Amay-Singhania"
 				(path "/94d2054e-a50f-482d-afff-dfa6248d499c"
-					(reference "#PWR038")
+					(reference "#PWR060")
 					(unit 1)
 				)
@@
 		(dnp no)
 		(fields_autoplaced yes)
-		(property "Reference" "#PWR031"
+		(property "Reference" "#PWR052"
 			(at 48.26 25.4 0)
 			(hide yes)
@@
 			(project "Amay-Singhania"
 				(path "/94d2054e-a50f-482d-afff-dfa6248d499c"
-					(reference "#PWR031")
+					(reference "#PWR052")
 					(unit 1)
 				)
@@
 		(dnp no)
 		(fields_autoplaced yes)
-		(property "Reference" "#PWR030"
+		(property "Reference" "#PWR051"
 			(at 40.64 53.34 0)
 			(hide yes)
@@
 			(project "Amay-Singhania"
 				(path "/94d2054e-a50f-482d-afff-dfa6248d499c"
-					(reference "#PWR030")
+					(reference "#PWR051")
 					(unit 1)
 				)
@@
 		(in_pos_files yes)
 		(dnp no)
-		(property "Reference" "#PWR035"
+		(property "Reference" "#PWR056"
 			(at 76.2 102.87 0)
 			(hide yes)
@@
 			(project "Amay-Singhania"
 				(path "/94d2054e-a50f-482d-afff-dfa6248d499c"
-					(reference "#PWR035")
+					(reference "#PWR056")
 					(unit 1)
 				)
@@
 		(in_pos_files yes)
 		(dnp no)
-		(property "Reference" "#PWR034"
+		(property "Reference" "#PWR055"
 			(at 73.66 113.03 0)
 			(hide yes)
@@
 			(project "Amay-Singhania"
 				(path "/94d2054e-a50f-482d-afff-dfa6248d499c"
-					(reference "#PWR034")
+					(reference "#PWR055")
 					(unit 1)
 				)
@@
 		(in_pos_files yes)
 		(dnp no)
-		(property "Reference" "#PWR039"
+		(property "Reference" "#PWR059"
 			(at 130.81 77.47 0)
 			(hide yes)
@@
 			(project "Amay-Singhania"
 				(path "/94d2054e-a50f-482d-afff-dfa6248d499c"
-					(reference "#PWR039")
+					(reference "#PWR059")
 					(unit 1)
 				)
@@
 		(in_pos_files yes)
 		(dnp no)
-		(property "Reference" "#PWR037"
+		(property "Reference" "#PWR058"
 			(at 106.68 113.03 0)
 			(hide yes)
@@
 			(project "Amay-Singhania"
 				(path "/94d2054e-a50f-482d-afff-dfa6248d499c"
-					(reference "#PWR037")
+					(reference "#PWR058")
 					(unit 1)
 				)
@@
 		(in_pos_files yes)
 		(dnp no)
-		(property "Reference" "#PWR032"
+		(property "Reference" "#PWR053"
 			(at 52.07 38.1 0)
 			(hide yes)
@@
 			(project "Amay-Singhania"
 				(path "/94d2054e-a50f-482d-afff-dfa6248d499c"
-					(reference "#PWR032")
+					(reference "#PWR053")
 					(unit 1)
 				)
@@
 		(in_pos_files yes)
 		(dnp no)
-		(property "Reference" "#PWR033"
+		(property "Reference" "#PWR054"
 			(at 55.88 36.83 0)
 			(hide yes)
@@
 			(project "Amay-Singhania"
 				(path "/94d2054e-a50f-482d-afff-dfa6248d499c"
-					(reference "#PWR033")
+					(reference "#PWR054")
 					(unit 1)
 				)
@@
 		(dnp no)
 		(fields_autoplaced yes)
-		(property "Reference" "SW3"
+		(property "Reference" "SW5"
 			(at 85.09 97.7899 90)
 			(show_name no)
@@
 			)
 		)
-		(property "Footprint" ""
+		(property "Footprint" "Button_Switch_SMD:SW_DIP_SPSTx04_Slide_6.7x11.72mm_W6.73mm_P2.54mm_LowProfile_JPin"
 			(at 76.2 99.06 0)
 			(hide yes)
@@
 			(project "Amay-Singhania"
 				(path "/94d2054e-a50f-482d-afff-dfa6248d499c"
-					(reference "SW3")
+					(reference "SW5")
 					(unit 1)
 				)
@@
 		(dnp no)
 		(fields_autoplaced yes)
-		(property "Reference" "C13"
+		(property "Reference" "C17"
 			(at 130.81 41.91 90)
 			(show_name no)
@@
 			)
 		)
-		(property "Footprint" "Package_TO_SOT_SMD:TSOT-23-5"
+		(property "Footprint" "Capacitor_SMD:C_0402_1005Metric"
 			(at 127 50.4952 0)
 			(hide yes)
@@
 			(project "Amay-Singhania"
 				(path "/94d2054e-a50f-482d-afff-dfa6248d499c"
-					(reference "C13")
+					(reference "C17")
 					(unit 1)
 				)
