File: lv/Amay-Singhania/strain_gauges.kicad_sch (KiCad schematic)
At the start: 20 parts, among them SW1 SW_DIP_x04, SW2 SW_DIP_x04, U1 ADS1119IRTER, U2 AD8222HACPZ-R7, U3 AD8222HACPZ-R7

Commit message: Updated PCB with RC values for low pass filter. has old onboarding sheets with in-Amp and other designs, will be removed in next commit
Parts:
- C10: renamed from C5; footprint Package_TO_SOT_SMD:TSOT-23-5 -> Capacitor_SMD:C_0402_1005Metric
- C11: renamed from C6; footprint Package_TO_SOT_SMD:TSOT-23-5 -> Capacitor_SMD:C_0402_1005Metric
- C12: renamed from C7; footprint Package_TO_SOT_SMD:TSOT-23-5 -> Capacitor_SMD:C_0402_1005Metric
- C13: renamed from C10; footprint Package_TO_SOT_SMD:TSOT-23-5 -> Capacitor_SMD:C_0402_1005Metric
- C14: renamed from C8; footprint Package_TO_SOT_SMD:TSOT-23-5 -> Capacitor_SMD:C_0402_1005Metric
- C4: renamed from C1; footprint Package_TO_SOT_SMD:TSOT-23-5 -> Capacitor_SMD:C_0402_1005Metric
- C5: renamed from C2; footprint Package_TO_SOT_SMD:TSOT-23-5 -> Capacitor_SMD:C_0402_1005Metric
- C6: renamed from C3; footprint Package_TO_SOT_SMD:TSOT-23-5 -> Capacitor_SMD:C_0402_1005Metric
- C7: renamed from C4; footprint Package_TO_SOT_SMD:TSOT-23-5 -> Capacitor_SMD:C_0402_1005Metric
- C8: renamed from C14; footprint Package_TO_SOT_SMD:TSOT-23-5 -> Capacitor_SMD:C_0402_1005Metric
- C9: footprint Package_TO_SOT_SMD:TSOT-23-5 -> Capacitor_SMD:C_0402_1005Metric
- R10: renamed from R22; footprint Package_DIP:DIP-8_W7.62mm -> Resistor_SMD:R_0402_1005Metric
- R7: footprint Package_DIP:DIP-8_W7.62mm -> Resistor_SMD:R_0402_1005Metric
- R8: renamed from R20; footprint Package_DIP:DIP-8_W7.62mm -> Resistor_SMD:R_0402_1005Metric
- R9: renamed from R21; footprint Package_DIP:DIP-8_W7.62mm -> Resistor_SMD:R_0402_1005Metric
- SW3: renamed from SW2; footprint RTE0016D -> Button_Switch_SMD:SW_DIP_SPSTx04_Slide_6.7x11.72mm_W6.73mm_P2.54mm_LowProfile_JPin
- SW4: renamed from SW1; footprint RTE0016D -> Button_Switch_SMD:SW_DIP_SPSTx04_Slide_6.7x11.72mm_W6.73mm_P2.54mm_LowProfile_JPin
- renumbered U1 to U3, U3 to U4
Connections:
- net +IN Center Axial Gauge renamed +IN Center_Gauge
- net +IN Left Axial Gauge renamed +IN Left_Gauge
- net +IN Right Axial Gauge renamed +IN Right_Gauge
- net -IN Center Axial Gauge renamed -IN Center_Gauge
- net -IN Left Axial Gauge renamed -IN Left_Gauge
- net -IN Right Axial Gauge renamed -IN Right_Gauge
- net ADC SCL renamed ADC_SCL
- net ADC SDA renamed ADC_SDA
- net Reference Gauge Out renamed Reference_Gauge_Out
