File: lv/Amay-Singhania/op-amp_buffer.kicad_sch (KiCad schematic)
At the start: 8 parts, among them SW3 SW_DIP_x04, SW4 SW_DIP_x02, U2 ADS122C14IRTER

Commit message: wjker
Parts:
- U1: renamed from U2; footprint RTE0016C-IPC_A -> ADS122C14:RTE0016C-IPC_A
- renumbered C5 to C10, C6 to C11, C4 to C9, JP3 to JP4, JP4 to JP5, SW3 to SW1, SW4 to SW2
Other:
- note added: "1140 + 92 + 4714.28571429 * 5 = ~24,803 uA = ~24mA ADC AVDD + ADC DVDD + Strain Gauges + Reference voltage divider = total current on 3V3"
Changed lines of the file:
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@@
+		)
+	)
+	(text "1140 + 92 + 4714.28571429 * 5 = ~24,803 uA = ~24mA\nADC AVDD + ADC DVDD + Strain Gauges + Reference voltage divider = total current on 3V3"
+		(exclude_from_sim no)
+		(at 127.508 128.778 0)
+		(effects
+			(font
+				(size 1.27 1.27)
+			)
 		)
 	)
@@
 	(wire
 		(pts
-			(xy 68.58 36.83) (xy 71.12 36.83)
+			(xy 66.04 36.83) (xy 68.58 36.83)
 		)
 		(stroke
@@
 	(wire
 		(pts
-			(xy 71.12 36.83) (xy 71.12 39.37)
+			(xy 66.04 36.83) (xy 66.04 39.37)
 		)
 		(stroke
@@
 		(dnp no)
 		(fields_autoplaced yes)
-		(property "Reference" "U2"
+		(property "Reference" "U1"
 			(at 124.46 40.64 0)
 			(show_name no)
@@
 			)
 		)
-		(property "Footprint" "RTE0016C-IPC_A"
+		(property "Footprint" "ADS122C14:RTE0016C-IPC_A"
 			(at 90.17 50.8 0)
 			(hide yes)
@@
 			(project "Amay-Singhania"
 				(path "/c320de66-ef76-480d-89b6-cc5374f65a42"
-					(reference "U2")
+					(reference "U1")
 					(unit 1)
 				)
@@
 		(in_pos_files yes)
 		(dnp no)
-		(property "Reference" "#PWR028"
+		(property "Reference" "#PWR035"
 			(at 173.99 58.42 0)
 			(hide yes)
@@
 			(project "Amay-Singhania"
 				(path "/c320de66-ef76-480d-89b6-cc5374f65a42"
-					(reference "#PWR028")
+					(reference "#PWR035")
 					(unit 1)
 				)
@@
 		(in_pos_files yes)
 		(dnp no)
-		(property "Reference" "C4"
-			(at 61.976 49.022 0)
+		(property "Reference" "C9"
+			(at 61.214 49.022 0)
 			(show_name no)
 			(do_not_autoplace no)
@@
 		)
 		(property "Value" "100nF"
-			(at 60.452 51.308 0)
+			(at 59.69 51.308 0)
 			(show_name no)
 			(do_not_autoplace no)
@@
 			(project "Amay-Singhania"
 				(path "/c320de66-ef76-480d-89b6-cc5374f65a42"
-					(reference "C4")
+					(reference "C9")
 					(unit 1)
 				)
@@
 		(in_pos_files yes)
 		(dnp no)
-		(property "Reference" "JP4"
+		(property "Reference" "JP5"
 			(at 65.278 73.66 90)
 			(show_name no)
@@
 			(project "Amay-Singhania"
 				(path "/c320de66-ef76-480d-89b6-cc5374f65a42"
-					(reference "JP4")
+					(reference "JP5")
 					(unit 1)
 				)
@@
 		(dnp no)
 		(fields_autoplaced yes)
-		(property "Reference" "SW4"
+		(property "Reference" "SW2"
 			(at 144.78 99.0599 90)
 			(show_name no)
@@
 			(project "Amay-Singhania"
 				(path "/c320de66-ef76-480d-89b6-cc5374f65a42"
-					(reference "SW4")
+					(reference "SW2")
 					(unit 1)
 				)
@@
 		(dnp no)
 		(fields_autoplaced yes)
-		(property "Reference" "C6"
+		(property "Reference" "C11"
 			(at 165.1 43.18 90)
 			(show_name no)
@@
 			(project "Amay-Singhania"
 				(path "/c320de66-ef76-480d-89b6-cc5374f65a42"
-					(reference "C6")
+					(reference "C11")
 					(unit 1)
 				)
@@
 		(in_pos_files yes)
 		(dnp no)
-		(property "Reference" "#PWR027"
+		(property "Reference" "#PWR034"
 			(at 167.64 83.82 0)
 			(hide yes)
@@
 			(project "Amay-Singhania"
 				(path "/c320de66-ef76-480d-89b6-cc5374f65a42"
-					(reference "#PWR027")
+					(reference "#PWR034")
 					(unit 1)
 				)
@@
 		(dnp no)
 		(fields_autoplaced yes)
-		(property "Reference" "SW3"
+		(property "Reference" "SW1"
 			(at 119.38 99.0599 90)
 			(show_name no)
@@
 			(project "Amay-Singhania"
 				(path "/c320de66-ef76-480d-89b6-cc5374f65a42"
-					(reference "SW3")
+					(reference "SW1")
 					(unit 1)
 				)
@@
 		(in_pos_files yes)
 		(dnp no)
-		(property "Reference" "C5"
+		(property "Reference" "C10"
 			(at 75.438 43.18 0)
 			(show_name no)
@@
 			(project "Amay-Singhania"
 				(path "/c320de66-ef76-480d-89b6-cc5374f65a42"
-					(reference "C5")
+					(reference "C10")
 					(unit 1)
 				)
@@
 		(in_pos_files yes)
 		(dnp no)
-		(property "Reference" "JP3"
+		(property "Reference" "JP4"
 			(at 61.722 63.5 90)
 			(show_name no)
@@
 			(project "Amay-Singhania"
 				(path "/c320de66-ef76-480d-89b6-cc5374f65a42"
-					(reference "JP3")
+					(reference "JP4")
 					(unit 1)
 				)
@@
 		(in_pos_files yes)
 		(dnp no)
-		(property "Reference" "#PWR026"
+		(property "Reference" "#PWR033"
 			(at 162.56 86.36 0)
 			(hide yes)
@@
 			(project "Amay-Singhania"
 				(path "/c320de66-ef76-480d-89b6-cc5374f65a42"
-					(reference "#PWR026")
+					(reference "#PWR033")
 					(unit 1)
 				)
@@
 		(in_pos_files yes)
 		(dnp no)
-		(property "Reference" "#PWR022"
+		(property "Reference" "#PWR027"
 			(at 78.74 40.64 0)
 			(hide yes)
@@
 			(project "Amay-Singhania"
 				(path "/c320de66-ef76-480d-89b6-cc5374f65a42"
-					(reference "#PWR022")
+					(reference "#PWR027")
 					(unit 1)
 				)
@@
 		(in_pos_files yes)
 		(dnp no)
-		(property "Reference" "#PWR023"
+		(property "Reference" "#PWR028"
 			(at 90.17 44.45 0)
 			(hide yes)
@@
 			(project "Amay-Singhania"
 				(path "/c320de66-ef76-480d-89b6-cc5374f65a42"
-					(reference "#PWR023")
+					(reference "#PWR028")
 					(unit 1)
 				)
@@
 		(in_pos_files yes)
 		(dnp no)
-		(property "Reference" "#PWR085"
+		(property "Reference" "#PWR031"
 			(at 133.35 113.03 0)
 			(hide yes)
@@
 			(project "Amay-Singhania"
 				(path "/c320de66-ef76-480d-89b6-cc5374f65a42"
-					(reference "#PWR085")
+					(reference "#PWR031")
 					(unit 1)
 				)
@@
 		(in_pos_files yes)
 		(dnp no)
-		(property "Reference" "#PWR025"
+		(property "Reference" "#PWR032"
 			(at 140.97 116.84 0)
 			(hide yes)
@@
 			(project "Amay-Singhania"
 				(path "/c320de66-ef76-480d-89b6-cc5374f65a42"
-					(reference "#PWR025")
+					(reference "#PWR032")
 					(unit 1)
 				)
@@
 		(in_pos_files yes)
 		(dnp no)
-		(property "Reference" "#PWR024"
+		(property "Reference" "#PWR030"
 			(at 110.49 118.11 0)
 			(hide yes)
@@
 			(project "Amay-Singhania"
 				(path "/c320de66-ef76-480d-89b6-cc5374f65a42"
-					(reference "#PWR024")
+					(reference "#PWR030")
 					(unit 1)
 				)
@@
 	(symbol
 		(lib_id "power:GND")
-		(at 71.12 39.37 0)
+		(at 66.04 39.37 0)
 		(unit 1)
 		(body_style 1)
@@
 		(in_pos_files yes)
 		(dnp no)
-		(property "Reference" "#PWR015"
-			(at 71.12 45.72 0)
+		(property "Reference" "#PWR026"
+			(at 66.04 45.72 0)
 			(hide yes)
 			(show_name no)
@@
 		)
 		(property "Value" "GND"
-			(at 71.12 43.434 0)
+			(at 66.04 43.434 0)
 			(show_name no)
 			(do_not_autoplace no)
@@
 		)
 		(property "Footprint" ""
-			(at 71.12 39.37 0)
+			(at 66.04 39.37 0)
 			(hide yes)
 			(show_name no)
@@
 		)
 		(property "Datasheet" ""
-			(at 71.12 39.37 0)
+			(at 66.04 39.37 0)
 			(hide yes)
 			(show_name no)
@@
 		)
 		(property "Description" "Power symbol creates a global label with name \"GND\" , ground"
-			(at 71.12 39.37 0)
+			(at 66.04 39.37 0)
 			(hide yes)
 			(show_name no)
@@
 			(project "Amay-Singhania"
 				(path "/c320de66-ef76-480d-89b6-cc5374f65a42"
-					(reference "#PWR015")
+					(reference "#PWR026")
 					(unit 1)
 				)
@@
 		(in_pos_files yes)
 		(dnp no)
-		(property "Reference" "#PWR075"
+		(property "Reference" "#PWR029"
 			(at 101.6 111.76 0)
 			(hide yes)
@@
 			(project "Amay-Singhania"
 				(path "/c320de66-ef76-480d-89b6-cc5374f65a42"
-					(reference "#PWR075")
+					(reference "#PWR029")
 					(unit 1)
 				)
@@
 		(dnp no)
 		(fields_autoplaced yes)
-		(property "Reference" "#PWR012"
+		(property "Reference" "#PWR025"
 			(at 57.15 54.61 0)
 			(hide yes)
@@
 			(project "Amay-Singhania"
 				(path "/c320de66-ef76-480d-89b6-cc5374f65a42"
-					(reference "#PWR012")
+					(reference "#PWR025")
 					(unit 1)
 				)

Commit message: added voltage regulators and finished schematic
Parts:
- U3: renamed from U1; footprint ADS122C14:RTE0016C-IPC_A -> RTE0016C-IPC_A
Changed lines of the file:
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@@
 		(dnp no)
 		(fields_autoplaced yes)
-		(property "Reference" "U1"
+		(property "Reference" "U3"
 			(at 124.46 40.64 0)
 			(show_name no)
@@
 			)
 		)
-		(property "Footprint" "ADS122C14:RTE0016C-IPC_A"
+		(property "Footprint" "RTE0016C-IPC_A"
 			(at 90.17 50.8 0)
 			(hide yes)
@@
 			(project "Amay-Singhania"
 				(path "/c320de66-ef76-480d-89b6-cc5374f65a42"
-					(reference "U1")
+					(reference "U3")
 					(unit 1)
 				)
@@
 		(in_pos_files yes)
 		(dnp no)
-		(property "Reference" "#PWR035"
+		(property "Reference" "#PWR037"
 			(at 173.99 58.42 0)
 			(hide yes)
@@
 			(project "Amay-Singhania"
 				(path "/c320de66-ef76-480d-89b6-cc5374f65a42"
-					(reference "#PWR035")
+					(reference "#PWR037")
 					(unit 1)
 				)
@@
 		(in_pos_files yes)
 		(dnp no)
-		(property "Reference" "#PWR034"
+		(property "Reference" "#PWR036"
 			(at 167.64 83.82 0)
 			(hide yes)
@@
 			(project "Amay-Singhania"
 				(path "/c320de66-ef76-480d-89b6-cc5374f65a42"
-					(reference "#PWR034")
+					(reference "#PWR036")
 					(unit 1)
 				)
@@
 		(in_pos_files yes)
 		(dnp no)
-		(property "Reference" "#PWR033"
+		(property "Reference" "#PWR035"
 			(at 162.56 86.36 0)
 			(hide yes)
@@
 			(project "Amay-Singhania"
 				(path "/c320de66-ef76-480d-89b6-cc5374f65a42"
-					(reference "#PWR033")
+					(reference "#PWR035")
 					(unit 1)
 				)
@@
 		(in_pos_files yes)
 		(dnp no)
-		(property "Reference" "#PWR027"
+		(property "Reference" "#PWR029"
 			(at 78.74 40.64 0)
 			(hide yes)
@@
 			(project "Amay-Singhania"
 				(path "/c320de66-ef76-480d-89b6-cc5374f65a42"
-					(reference "#PWR027")
+					(reference "#PWR029")
 					(unit 1)
 				)
@@
 		(in_pos_files yes)
 		(dnp no)
-		(property "Reference" "#PWR028"
+		(property "Reference" "#PWR030"
 			(at 90.17 44.45 0)
 			(hide yes)
@@
 			(project "Amay-Singhania"
 				(path "/c320de66-ef76-480d-89b6-cc5374f65a42"
-					(reference "#PWR028")
+					(reference "#PWR030")
 					(unit 1)
 				)
@@
 		(in_pos_files yes)
 		(dnp no)
-		(property "Reference" "#PWR031"
+		(property "Reference" "#PWR033"
 			(at 133.35 113.03 0)
 			(hide yes)
@@
 			(project "Amay-Singhania"
 				(path "/c320de66-ef76-480d-89b6-cc5374f65a42"
-					(reference "#PWR031")
+					(reference "#PWR033")
 					(unit 1)
 				)
@@
 		(in_pos_files yes)
 		(dnp no)
-		(property "Reference" "#PWR032"
+		(property "Reference" "#PWR034"
 			(at 140.97 116.84 0)
 			(hide yes)
@@
 			(project "Amay-Singhania"
 				(path "/c320de66-ef76-480d-89b6-cc5374f65a42"
-					(reference "#PWR032")
+					(reference "#PWR034")
 					(unit 1)
 				)
@@
 		(in_pos_files yes)
 		(dnp no)
-		(property "Reference" "#PWR030"
+		(property "Reference" "#PWR032"
 			(at 110.49 118.11 0)
 			(hide yes)
@@
 			(project "Amay-Singhania"
 				(path "/c320de66-ef76-480d-89b6-cc5374f65a42"
-					(reference "#PWR030")
+					(reference "#PWR032")
 					(unit 1)
 				)
@@
 		(in_pos_files yes)
 		(dnp no)
-		(property "Reference" "#PWR026"
+		(property "Reference" "#PWR028"
 			(at 66.04 45.72 0)
 			(hide yes)
@@
 			(project "Amay-Singhania"
 				(path "/c320de66-ef76-480d-89b6-cc5374f65a42"
-					(reference "#PWR026")
+					(reference "#PWR028")
 					(unit 1)
 				)
@@
 		(in_pos_files yes)
 		(dnp no)
-		(property "Reference" "#PWR029"
+		(property "Reference" "#PWR031"
 			(at 101.6 111.76 0)
 			(hide yes)
@@
 			(project "Amay-Singhania"
 				(path "/c320de66-ef76-480d-89b6-cc5374f65a42"
-					(reference "#PWR029")
+					(reference "#PWR031")
 					(unit 1)
 				)
@@
 		(dnp no)
 		(fields_autoplaced yes)
-		(property "Reference" "#PWR025"
+		(property "Reference" "#PWR027"
 			(at 57.15 54.61 0)
 			(hide yes)
@@
 			(project "Amay-Singhania"
 				(path "/c320de66-ef76-480d-89b6-cc5374f65a42"
-					(reference "#PWR025")
-					(unit 1)
-				)
+					(reference "#PWR027")
+					(unit 1)
+				)

Commit message: final commit to onboarding, moved to fpc-strain-gauge in fs-5-schematics repo
Connections:
- net Address Pin 2: now reaches SW2.1, SW2.2, U3.10 (A1)
- net Address Pin 1: now reaches SW1.1, SW1.2, SW1.3, SW1.4, U3.9 (A0)
Changed lines of the file:
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@@
+		)
+	)
+	(label "Address Pin 1"
+		(at 149.86 87.63 0)
+		(effects
+			(font
+				(size 1.27 1.27)
+			)
+			(justify left bottom)
+		)
+	)
+	(label "Address Pin 2"
+		(at 149.86 90.17 0)
+		(effects
+			(font
+				(size 1.27 1.27)
+			)
+			(justify left bottom)
 		)
 	)
